Commit message: satellite080919

File: hector_quadrotor/hector_quadrotor_description/urdf/quadrotor_base.urdf.xacro (robot description, xacro)
@@ -21,4 +21,7 @@
         <origin xyz="0 0 0" rpy="0 0 0" />
         <geometry>
+          <box>
+            <size>0.3 0.3 0.01</size>
+          </box>
           <mesh filename="package://hector_quadrotor_description/meshes/quadrotor/quadrotor_base.stl"/>
         </geometry>

Commit message: 260919

File: hector_quadrotor/hector_quadrotor_description/urdf/quadrotor_base.urdf.xacro (robot description, xacro)
@@ -21,7 +21,4 @@
         <origin xyz="0 0 0" rpy="0 0 0" />
         <geometry>
-          <box>
-            <size>0.3 0.3 0.01</size>
-          </box>
           <mesh filename="package://hector_quadrotor_description/meshes/quadrotor/quadrotor_base.stl"/>
         </geometry>

File: hector_quadrotor/hector_quadrotor_description/urdf/quadrotor_hokuyo_utm30lx.urdf.xacro (robot description, xacro)
@@ -12,7 +12,12 @@
     </xacro:hokuyo_utm30lx>
     <!-- Forward facing camera -->
-    <xacro:include filename="$(find hector_sensors_description)/urdf/generic_camera.urdf.xacro" />
+    <!--<xacro:include filename="$(find hector_sensors_description)/urdf/generic_camera.urdf.xacro" />
     <xacro:generic_camera name="front_cam" parent="base_link" ros_topic="camera/image" cam_info_topic="camera/camera_info" update_rate="10" res_x="320" res_y="240" image_format="R8G8B8" hfov="90">
       <origin xyz="0.05 0.0 -0.06" rpy="0 0 0"/>
+    </xacro:generic_camera>-->
+    <!-- Downward facing camera -->
+    <xacro:include filename="$(find hector_sensors_description)/urdf/generic_camera.urdf.xacro" />
+    <xacro:generic_camera name="downward_cam" parent="base_link" ros_topic="camera/image" cam_info_topic="camera/camera_info" update_rate="20" res_x="640" res_y="480" image_format="L8" hfov="100">
+      <origin xyz="0.4 0.0 -0.0" rpy="0 ${M_PI/2} 0"/>
     </xacro:generic_camera>
 </robot>
